File: .claude/skills/kicad-schematic-gen/evals/corpus/synthetic/battery_3s_full/golden.kicad_sch (KiCad schematic)
At the start: 74 parts, among them J1 USB-C, J2 JST-PH 2-pin, J4 JST-PH 2-pin, J5 JST-PH 2-pin, J6 JST-PH 3-pin, J7 JST-PH 2-pin, Q1 AO4407A, Q6 AO4407A, Q7 AO3400A, Q8 AO3400A, Q9 AO3400A, U1 CH224K, U2 MAX77961EFV06+, U3 AP63200WU-7, U6 USBLC6-2SC6

Commit message: updated bom handling within kicad
Parts:
- C1, C17, C2, C3: MPN (none) -> CL32B106KBJNNNE; Manufacturer (none) -> Samsung; Package (none) -> 1210
- C10, C11: MPN (none) -> CL05B224KO5NNNC; Manufacturer (none) -> Samsung; Package (none) -> 0402
- C12, C13: MPN (none) -> CL21A475KAQNNNE; Manufacturer (none) -> Samsung; Package (none) -> 0805
- C14, C15: MPN (none) -> CL05B104KO5NNNC; Manufacturer (none) -> Samsung; Package (none) -> 0402
- C16, C20, C22, C4: MPN (none) -> CL21B104KBCNNNC; Manufacturer (none) -> Samsung; Package (none) -> 0805
- C18, C19: MPN (none) -> CL21A226MAYNNNE; Manufacturer (none) -> Samsung; Package (none) -> 0805
- C21, C8, C9: MPN (none) -> CL21A106KAYNNNE; Manufacturer (none) -> Samsung; Package (none) -> 0805
- C23: MPN (none) -> CL05B103KO5NNNC; Manufacturer (none) -> Samsung; Package (none) -> 0402
- C5, C6, C7: MPN (none) -> GRM32ER61E476ME15L; Manufacturer (none) -> Murata; Package (none) -> 1210
- D1: MPN (none) -> 150080GS75000; Manufacturer (none) -> Wurth; Package (none) -> 0805
- D2: MPN (none) -> 150080RS75000; Manufacturer (none) -> Wurth; Package (none) -> 0805
- D3, D8: MPN (none) -> SMF15A; Manufacturer (none) -> Littelfuse; Package (none) -> SOD-123FL
- D7: MPN (none) -> SS34; Manufacturer (none) -> Diodes Inc; Package (none) -> SMA
- J1: MPN (none) -> USB4125-GF-A; Manufacturer (none) -> GCT; Package (none) -> USB-C
- J2, J4, J5, J7: MPN (none) -> S2B-PH-SM4-TB(LF)(SN); Manufacturer (none) -> JST; Package (none) -> JST-PH
- J6: MPN (none) -> S3B-PH-SM4-TB(LF)(SN); Manufacturer (none) -> JST; Package (none) -> JST-PH
- L1: MPN (none) -> SWPA6045S3R3NT; Manufacturer (none) -> Sunlord; Package (none) -> SWPA6045
- L2: MPN (none) -> CYA0630-4R7M; Manufacturer (none) -> Chilisin; Package (none) -> CYA0630
- Q1, Q6: MPN (none) -> AO4407A; Manufacturer (none) -> Alpha & Omega; Package (none) -> SOIC-8
- Q7, Q8, Q9: MPN (none) -> AO3400A; Manufacturer (none) -> Alpha & Omega; Package (none) -> SOT-23
- R1: MPN (none) -> RC0805FR-0756KL; Manufacturer (none) -> YAGEO; Package (none) -> 0805
- R10, R12, R13, R14, R18, R2, R8: MPN (none) -> RC0805FR-0710KL; Manufacturer (none) -> YAGEO; Package (none) -> 0805
- R11: MPN (none) -> RC0805FR-07200KL; Manufacturer (none) -> YAGEO; Package (none) -> 0805
- R15, R16: MPN (none) -> RC0805FR-0710RL; Manufacturer (none) -> YAGEO; Package (none) -> 0805
- R17: MPN (none) -> RC0805FR-0752K3L; Manufacturer (none) -> YAGEO; Package (none) -> 0805
- R19, R20: MPN (none) -> RC0805FR-071KL; Manufacturer (none) -> YAGEO; Package (none) -> 0805
- R21, R22, R24, R25, R27: MPN (none) -> RC0805FR-07100KL; Manufacturer (none) -> YAGEO; Package (none) -> 0805
- R23: MPN (none) -> RC0805FR-071ML; Manufacturer (none) -> YAGEO; Package (none) -> 0805
- R26: MPN (none) -> RC0805FR-07470KL; Manufacturer (none) -> YAGEO; Package (none) -> 0805
- R3: MPN (none) -> RC0805FR-078K66L; Manufacturer (none) -> YAGEO; Package (none) -> 0805
- R4: MPN (none) -> RC0805FR-07178KL; Manufacturer (none) -> YAGEO; Package (none) -> 0805
- R5: MPN (none) -> RC0805FR-0754K9L; Manufacturer (none) -> YAGEO; Package (none) -> 0805
- R6: MPN (none) -> RC0805FR-0714KL; Manufacturer (none) -> YAGEO; Package (none) -> 0805
- R7: MPN (none) -> RC0805FR-07226KL; Manufacturer (none) -> YAGEO; Package (none) -> 0805
- R9: MPN (none) -> RC0805FR-074R7L; Manufacturer (none) -> YAGEO; Package (none) -> 0805
- RS1: MPN (none) -> WSL1206R0100FEA; Manufacturer (none) -> Vishay; Package (none) -> 1206
- RT1: MPN (none) -> NCP15XH103F03RC; Manufacturer (none) -> Murata; Package (none) -> 0805
- U1: MPN (none) -> CH224K; Manufacturer (none) -> WCH; Package (none) -> SSOP-10
- U2: MPN (none) -> MAX77961EFV06+; Manufacturer (none) -> Analog Devices; Package (none) -> FC2QFN-30
- U3: MPN (none) -> AP63200WU-7; Manufacturer (none) -> Diodes Inc; Package (none) -> TSOT-23-6
- U6: MPN (none) -> USBLC6-2SC6; Manufacturer (none) -> STMicroelectronics; Package (none) -> SOT-23-6
