File: .claude/skills/kicad-schematic-gen/tests/fixtures/battery_3s/battery_3s.golden.kicad_sch (KiCad schematic)
At the start: 58 parts, among them J1 USB-C, J2 JST-PH 2-pin, J4 JST-PH 2-pin, J5 JST-PH 2-pin, J6 1x3 header, J7 JST-PH 2-pin, Q1 AO3401A, Q2 AO3400A, Q3 AO3400A, Q4 AO3401A, U1 CH224K, U2 BQ24650, U3 TPS54202DDCR, U4 LTC4412ES6

Commit message: updated bom handling within kicad
Parts:
- C1, C10, C13, C14, C7, C8: MPN (none) -> CL21A106KAYNNNE; Manufacturer (none) -> Samsung; Package (none) -> 0805
- C11, C12, C15, C17, C19, C2, C3, C9: MPN (none) -> CL21B104KBCNNNC; Manufacturer (none) -> Samsung; Package (none) -> 0805
- C16: MPN (none) -> CL21B103KBCNNNC; Manufacturer (none) -> Samsung; Package (none) -> 0805
- C18, C4, C6: MPN (none) -> CL21B105KBFNNNE; Manufacturer (none) -> Samsung; Package (none) -> 0805
- C5: MPN (none) -> CL21B473KBCNNNC; Manufacturer (none) -> Samsung; Package (none) -> 0805
- D1: MPN (none) -> 150080GS75000; Manufacturer (none) -> Wurth; Package (none) -> 0805
- D2: MPN (none) -> 150080RS75000; Manufacturer (none) -> Wurth; Package (none) -> 0805
- F1: MPN (none) -> 1812L300THPR; Manufacturer (none) -> Littelfuse; Package (none) -> 1812
- J1: MPN (none) -> USB4125-GF-A; Manufacturer (none) -> GCT; Package (none) -> USB-C
- J2, J4, J5, J7: MPN (none) -> S2B-PH-K-S(LF)(SN); Manufacturer (none) -> JST; Package (none) -> JST-PH
- J6: MPN (none) -> 61300311121; Manufacturer (none) -> Wurth; Package (none) -> 1x03-2.54
- L1: MPN (none) -> MWSA0503S-100MT; Manufacturer (none) -> Sunlord; Package (none) -> MWSA0503
- L2: MPN (none) -> MWSA0402S-100MT; Manufacturer (none) -> Sunlord; Package (none) -> MWSA0402
- Q1, Q4: MPN (none) -> AO3401A; Manufacturer (none) -> Alpha & Omega; Package (none) -> SOT-23
- Q2, Q3: MPN (none) -> AO3400A; Manufacturer (none) -> Alpha & Omega; Package (none) -> SOT-23
- R1: MPN (none) -> RC0805FR-0756KL; Manufacturer (none) -> YAGEO; Package (none) -> 0805
- R10, R12, R20, R7: MPN (none) -> RC0805FR-07100KL; Manufacturer (none) -> YAGEO; Package (none) -> 0805
- R11: MPN (none) -> RC0805FR-0713K3L; Manufacturer (none) -> YAGEO; Package (none) -> 0805
- R13, R14, R15, R9: MPN (none) -> RC0805FR-0710KL; Manufacturer (none) -> YAGEO; Package (none) -> 0805
- R16, R17: MPN (none) -> RC0805FR-071KL; Manufacturer (none) -> YAGEO; Package (none) -> 0805
- R19: MPN (none) -> RC0805FR-071ML; Manufacturer (none) -> YAGEO; Package (none) -> 0805
- R23, R24: MPN (none) -> RC0805FR-0710RL; Manufacturer (none) -> YAGEO; Package (none) -> 0805
- R4: MPN (none) -> RC0805FR-07953KL; Manufacturer (none) -> YAGEO; Package (none) -> 0805
- R5: MPN (none) -> RC0805FR-07200KL; Manufacturer (none) -> YAGEO; Package (none) -> 0805
- R6: MPN (none) -> RC0805FR-071M1L; Manufacturer (none) -> YAGEO; Package (none) -> 0805
- R8: MPN (none) -> RL1206FR-070R03L; Manufacturer (none) -> YAGEO; Package (none) -> 1206
- RT1: MPN (none) -> NCP15XH103F03RC; Manufacturer (none) -> Murata; Package (none) -> 0805
- U1: MPN (none) -> CH224K; Manufacturer (none) -> WCH; Package (none) -> SSOP-10
- U2: MPN (none) -> BQ24650RVAR; Manufacturer (none) -> Texas Instruments; Package (none) -> VQFN-16
- U3: MPN (none) -> TPS54202DDCR; Manufacturer (none) -> Texas Instruments; Package (none) -> SOT-23-6
- U4: MPN (none) -> LTC4412ES6#TRPBF; Manufacturer (none) -> Analog Devices; Package (none) -> TSOT-23-6
